File: schematic_board/kicad(latest)/schema.kicad_sch (KiCad schematic)
At the start: 29 parts, among them IC1 TLC271CPS, IC2 LM311D, Q1 IRLML6244TRPBF

Commit message: Latest schematic and board design
Parts:
- IC1: footprint SamacSys_Parts:SOIC127P780X200-8N -> Package_SO:SOIC-8_3.9x4.9mm_P1.27mm
Changed lines of the file:
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@@
 			)
 		)
-		(property "Footprint" "SamacSys_Parts:SOIC127P780X200-8N"
+		(property "Footprint" "Package_SO:SOIC-8_3.9x4.9mm_P1.27mm"
 			(at 107.95 224.46 0)
 			(effects
